Commit message: New update 19.03

File: description/robot.urdf.xacro (robot description, xacro)
@@ -2,4 +2,6 @@
 <robot xmlns:xacro="http://www.ros.org/wiki/xacro"  name="robot">
     <xacro:include filename="robot_core.xacro" />
-    <xacro:include filename="gazebo_control.xacro"/>
+    <!-- <xacro:include filename="gazebo_control.xacro"/> -->
+     <xacro:include filename="lidar.xacro"/>
+     <xacro:include filename="ros2_control.xacro"/>
 </robot>

File: description/robot_core.xacro (robot description, xacro)
@@ -14,4 +14,7 @@
   <material name = "black">
   <color rgba = "0 0 0 1"/>
+  </material>
+  <material name = "red">
+  <color rgba = "1 0 0 1"/>
   </material>
 <!--making out links-->

Commit message: Update 22.03

File: description/robot.urdf.xacro (robot description, xacro)
@@ -1,7 +1,7 @@
 <?xml version="1.0"?>
 <robot xmlns:xacro="http://www.ros.org/wiki/xacro"  name="robot">
+<xacro:include filename = "ros2_control.xacro"/>
     <xacro:include filename="robot_core.xacro" />
     <!-- <xacro:include filename="gazebo_control.xacro"/> -->
      <xacro:include filename="lidar.xacro"/>
-     <xacro:include filename="ros2_control.xacro"/>
 </robot>

File: description/robot_core.xacro (robot description, xacro)
@@ -20,4 +20,11 @@
 <!--making out links-->
 <link name = "base_link">
+</link>
+<joint name="base_footprint_joint" type="fixed">
+<parent link="base_link"/>
+<child link="base_footprint"/>
+<origin  xyz="0 0 0" rpy="0 0 0"/>
+</joint>
+<link name = "base_footprint">
 </link>
 <!--making joint-->

File: description/ros2_control.xacro (robot description, xacro)
@@ -21,4 +21,6 @@
             <state_interface name="position"/>
         </joint>
+        <!-- <odometry_frame>odom</odometry_frame>
+        <robot_base_frame>base_link</robot_base_frame> -->
     </ros2_control>
     <gazebo>
