Commit message: 26.03

File: description/lidar.xacro (robot description, xacro)
@@ -5,5 +5,5 @@
 <parent link="chassis"/>
 <child link = "laser_frame"/>
-<origin xyz="0.1 0 0.175 " rpy="0 0 0"/>
+<origin xyz="0.122 0 0.212" rpy="0 0 0"/>
 </joint>
  <!--link-->
@@ -15,4 +15,11 @@
 <material name="red"/>
 </visual>
+ <visual>
+<origin xyz="0 0 -0.05"/>
+<geometry>
+<cylinder radius="0.01" length="0.1"/>
+</geometry>
+ <material name="red"/>
+  </visual>
 <!--collision-->
 <collision>
@@ -35,4 +42,5 @@
                     <horizontal>
                         <samples>360</samples>
+                        <resolution>1</resolution>
                         <min_angle>-3.14</min_angle>
                         <max_angle>3.14</max_angle>
@@ -42,4 +50,5 @@
                     <min>0.3</min>
                     <max>12</max>
+                    <resolution>0.01</resolution>
                 </range>
             </ray>

File: description/robot_core.xacro (robot description, xacro)
@@ -90,5 +90,5 @@
 <parent link= "base_link"/>
 <child link = "right_wheel"/>
-<origin xyz="0 -0.175 0" rpy="${-pi/2} 0 0"/>
+<origin xyz="0 -0.175 0" rpy="${pi/2} 0 0"/>
 <axis xyz="0 0 -1"/>
 </joint>

File: description/ros2_control.xacro (robot description, xacro)
@@ -2,26 +2,24 @@
 <robot xmlns:xacro="http://www.ros.org/wiki/xacro">
     <ros2_control name="GazeboSystem" type="system">
-        <hardware>
-            <plugin>gazebo_ros2_control/GazeboSystem</plugin>
-        </hardware>
-        <joint name="left_wheel_joint">
-            <command_interface name="velocity">
-                <param name="min">-10</param>
-                <param name="max">10</param>
-            </command_interface>
-            <state_interface name="velocity"/>
-            <state_interface name="position"/>
-        </joint>
-        <joint name="right_wheel_joint">
-            <command_interface name="velocity">
-                <param name="min">-10</param>
-                <param name="max">10</param>
-            </command_interface>
-            <state_interface name="velocity"/>
-            <state_interface name="position"/>
-        </joint>
-        <!-- <odometry_frame>odom</odometry_frame>
-        <robot_base_frame>base_link</robot_base_frame> -->
-    </ros2_control>
+            <hardware>
+                <plugin>gazebo_ros2_control/GazeboSystem</plugin>
+            </hardware>
+            <joint name="left_wheel_joint">
+                <command_interface name="velocity">
+                    <param name="min">-10</param>
+                    <param name="max">10</param>
+                </command_interface>
+                <state_interface name="velocity"/>
+                <state_interface name="position"/>
+            </joint>
+            <joint name="right_wheel_joint">
+                <command_interface name="velocity">
+                    <param name="min">-10</param>
+                    <param name="max">10</param>
+                </command_interface>
+                <state_interface name="velocity"/>
+                <state_interface name="position"/>
+            </joint>
+        </ros2_control>
     <gazebo>
         <plugin name="gazebo_ros2_control" filename="libgazebo_ros2_control.so">
